File: ESP8266_thermostat.sch (KiCad schematic (older format))
At the start: 5 parts, among them Q1 2N2219, U1 DHT11, U2 WeMos_mini

Commit message: edits to IR circuit and DHT11 circuit
Parts:
- added R2: 10K, symbol Device:R_US
- R1: value R_US -> 47
Connections:
- net DHT11: now also R2.1; no longer U1.2 (IO)
- new net: R2.2, U1.2 (IO)
Changed lines of the file:
@@
 EESchema Schematic File Version 4
+LIBS:ESP8266_thermostat-cache
 EELAYER 26 0
 EELAYER END
@@
 Text Label 5900 3000 2    50   ~ 0
 DHT11
-Text Label 7000 2750 2    50   ~ 0
+Text Label 7100 2750 0    50   ~ 0
 DHT11
 $Comp
@@
 	6300 2400 6300 2450
 Wire Wire Line
-	6700 2750 7000 2750
-Wire Wire Line
 	5600 3000 5900 3000
-Text Label 3500 2950 0    50   ~ 0
+Text Label 3400 2950 0    50   ~ 0
 IR
 Text Label 4450 3000 0    50   ~ 0
@@
 Wire Wire Line
 	4450 3000 4600 3000
-Wire Wire Line
-	3500 2950 3600 2950
 NoConn ~ 5600 2700
 NoConn ~ 5600 2800
@@
 P 3900 3350
 F 0 "R1" H 3968 3396 50  0000 L CNN
-F 1 "R_US" H 3968 3305 50  0000 L CNN
+F 1 "47" H 3968 3305 50  0000 L CNN
 F 2 "" V 3940 3340 50  0001 C CNN
 F 3 "~" H 3900 3350 50  0001 C CNN
@@
 Wire Wire Line
 	3900 2400 3900 2350
+$Comp
+L Device:R_US R2
+U 1 1 5D4CC165
+P 6900 2750
+F 0 "R2" H 6968 2796 50  0000 L CNN
+F 1 "10K" H 6968 2705 50  0000 L CNN
+F 2 "" V 6940 2740 50  0001 C CNN
+F 3 "~" H 6900 2750 50  0001 C CNN
+	1    6900 2750
+	0    1    1    0
+$EndComp
+Wire Wire Line
+	7100 2750 7050 2750
+Wire Wire Line
+	6750 2750 6700 2750
+Wire Wire Line
+	3400 2950 3600 2950
 $EndSCHEMATC

Commit message: rescued symbols
Parts:
- Q1: symbol Transistor_BJT_2:2N2219 -> ESP8266_thermostat-rescue:2N2219-Transistor_BJT_2
- U1: symbol Sensor:DHT11 -> ESP8266_thermostat-rescue:DHT11-Sensor
- U2: symbol wemos_mini:WeMos_mini -> ESP8266_thermostat-rescue:WeMos_mini-wemos_mini
Changed lines of the file:
@@
 EESchema Schematic File Version 4
 LIBS:ESP8266_thermostat-cache
-EELAYER 26 0
+EELAYER 30 0
 EELAYER END
 $Descr A4 11693 8268
@@
 $EndDescr
 $Comp
-L wemos_mini:WeMos_mini U2
+L ESP8266_thermostat-rescue:WeMos_mini-wemos_mini U2
 U 1 1 5D4BA14C
 P 5100 2950
@@
 	5800 2600 5600 2600
 $Comp
-L Sensor:DHT11 U1
+L ESP8266_thermostat-rescue:DHT11-Sensor U1
 U 1 1 5D4BA646
 P 6400 2750
@@
 NoConn ~ 4600 3300
 $Comp
-L Transistor_BJT_2:2N2219 Q1
+L ESP8266_thermostat-rescue:2N2219-Transistor_BJT_2 Q1
 U 1 1 5D4BB904
 P 3800 2950
